File: electronics/reward_port/reward_port.kicad_pcb (KiCad board)
At the start: 4 copper layers, 30 x 40 mm, 61 parts, among them J1 SM04B-GHS-TB, J2 SM10B-GHS-TB, J3 SM10B-GHS-TB, J4 SM04B-GHS-TB, J5 Conn_SWD, J6 SM02B-GHS-TB, J7 SM02B-GHS-TB, Q1 2N7002, Q2 2N7002, Q3 2N7002, Q4 2N7002, U1 THVD1410DGKR, U2 THVD1410DGKR, U3 PAM8302AASCR, U4 STM32G071GBU6, U5 DRV8837

Commit message: small update to exact bulk capacitor, peripheral order list
Parts:
- C18: footprint Capacitor_Tantalum_SMD:CP_EIA-7360-38_Kemet-E -> Capacitor_Tantalum_SMD:CP_EIA-7343-43_Kemet-X
- Q1, Q2, Q3, Q4: value 2N7002 -> 2N7002PW
Changed lines of the file:
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@@
 			)
 		)
-		(property "Value" "2N7002"
+		(property "Value" "2N7002PW"
 			(at 0 1.8 90)
 			(layer "F.Fab")
@@
 			)
 		)
-		(property "Value" "2N7002"
+		(property "Value" "2N7002PW"
 			(at 0 1.8 90)
 			(layer "F.Fab")
@@
 			)
 		)
-		(property "Value" "2N7002"
+		(property "Value" "2N7002PW"
 			(at 0 1.8 90)
 			(layer "F.Fab")
@@
 			)
 		)
-		(property "Value" "2N7002"
+		(property "Value" "2N7002PW"
 			(at 0 1.8 90)
 			(layer "F.Fab")
@@
 		)
 	)
-	(footprint "Capacitor_Tantalum_SMD:CP_EIA-7360-38_Kemet-E"
+	(footprint "Capacitor_Tantalum_SMD:CP_EIA-7343-43_Kemet-X"
 		(layer "F.Cu")
 		(at 149.7 106.2 -90)
-		(descr "Tantalum Capacitor SMD Kemet-E (7360-38 Metric), IPC-7352 nominal, (Body size from: http://www.kemet.com/Lists/ProductCatalog/Attachments/253/KEM_TC101_STD.pdf)")
+		(descr "Tantalum Capacitor SMD Kemet-X (7343-43 Metric), IPC-7352 nominal, (Body size from: http://www.kemet.com/Lists/ProductCatalog/Attachments/253/KEM_TC101_STD.pdf)")
 		(tags "capacitor tantalum")
 		(property "Reference" "C18"
-			(at 0 -3.95 90)
+			(at 0 -3.1 270)
 			(layer "F.SilkS")
-			(hide yes)
 			(effects
 				(font
@@
 		)
 		(property "Value" "470uF"
-			(at 0 3.95 90)
+			(at 0 3.1 270)
 			(layer "F.Fab")
-			(hide yes)
 			(effects
 				(font
@@
 		)
 		(property "Datasheet" "EEEFP1A471AP"
-			(at 0 0 90)
+			(at 0 0 270)
 			(layer "F.Fab")
 			(hide yes)
@@
 		)
 		(property "Description" "Polarized capacitor"
-			(at 0 0 90)
+			(at 0 0 270)
 			(layer "F.Fab")
 			(hide yes)
@@
 		)
 		(property "KiLib_Generator" "SMD_2terminal_chip_molded"
-			(at 0 0 90)
+			(at 0 0 270)
 			(layer "F.SilkS")
 			(hide yes)
@@
 		(duplicate_pad_numbers_are_jumpers no)
 		(fp_line
-			(start -4.415 3.11)
-			(end 3.65 3.11)
+			(start -4.415 2.26)
+			(end 3.65 2.26)
 			(stroke
 				(width 0.12)
@@
 		)
 		(fp_line
-			(start -4.415 -3.11)
-			(end -4.415 3.11)
+			(start -4.415 -2.26)
+			(end -4.415 2.26)
 			(stroke
 				(width 0.12)
@@
 		)
 		(fp_line
-			(start 3.65 -3.11)
-			(end -4.415 -3.11)
+			(start 3.65 -2.26)
+			(end -4.415 -2.26)
 			(stroke
 				(width 0.12)
@@
 		)
 		(fp_rect
-			(start -4.41 -3.25)
-			(end 4.41 3.25)
+			(start -4.41 -2.4)
+			(end 4.41 2.4)
 			(stroke
 				(width 0.05)
@@
 		)
 		(fp_line
-			(start -3.65 3)
-			(end 3.65 3)
+			(start -3.65 2.15)
+			(end 3.65 2.15)
 			(stroke
 				(width 0.1)
@@
 		)
 		(fp_line
-			(start 3.65 3)
-			(end 3.65 -3)
+			(start 3.65 2.15)
+			(end 3.65 -2.15)
 			(stroke
 				(width 0.1)
@@
 		)
 		(fp_line
-			(start -3.65 -2)
-			(end -3.65 3)
+			(start -3.65 -1.15)
+			(end -3.65 2.15)
 			(stroke
 				(width 0.1)
@@
 		)
 		(fp_line
-			(start -2.65 -3)
-			(end -3.65 -2)
+			(start -2.65 -2.15)
+			(end -3.65 -1.15)
 			(stroke
 				(width 0.1)
@@
 		)
 		(fp_line
-			(start 3.65 -3)
-			(end -2.65 -3)
+			(start 3.65 -2.15)
+			(end -2.65 -2.15)
 			(stroke
 				(width 0.1)
@@
 		)
 		(fp_text user "${REFERENCE}"
-			(at 0 0 90)
+			(at 0 0 270)
 			(layer "F.Fab")
 			(effects
@@
 		(pad "1" smd roundrect
 			(at -3.12 0 270)
-			(size 2.07 4.29)
+			(size 2.07 2.59)
 			(layers "F.Cu" "F.Mask" "F.Paste")
 			(roundrect_rratio 0.120773)
@@
 		(pad "2" smd roundrect
 			(at 3.12 0 270)
-			(size 2.07 4.29)
+			(size 2.07 2.59)
 			(layers "F.Cu" "F.Mask" "F.Paste")
 			(roundrect_rratio 0.120773)
@@
 		)
 		(embedded_fonts no)
-		(model "${KICAD10_3DMODEL_DIR}/Capacitor_Tantalum_SMD.3dshapes/CP_EIA-7360-38_Kemet-E.step"
+		(model "${KICAD10_3DMODEL_DIR}/Capacitor_Tantalum_SMD.3dshapes/CP_EIA-7343-43_Kemet-X.step"
 			(offset
 				(xyz 0 0 0)
