File: electronics/head_sensor/head_sensor.kicad_sch (KiCad schematic)
At the start: 16 parts, among them J1 A79608-001, Q1 DMN2991UFB4, U1 LTC4332IUFD-PBF, U2 LSM6DSV32XTR, U3 MMC5983MA

Commit message: jlcpcb order for the head sensor
Parts:
- Q1: value DMN2991UFB4 -> DMN2300UFB4-7B
Changed lines of the file:
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@@
 			)
 		)
-		(property "Value" "DMN2991UFB4"
+		(property "Value" "DMN2300UFB4-7B"
 			(at 264.16 76.2 90)
 			(show_name no)
