File: electronics/head_sensor/head_sensor.kicad_pcb (KiCad board)
At the start: 4 copper layers, 9.8 x 7.6 mm, 16 parts, among them J1 A79608-001, Q1 DMN2991UFB4, U1 LTC4332IUFD-PBF, U2 LSM6DSV32XTR, U3 MMC5983MA

Commit message: Switching the transistor on floating hub to what was actually ordered
Parts:
- Q1: value DMN2991UFB4 -> DMN2300UFB4-7B
Changed lines of the file:
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@@
 			(outputformat 1)
 			(mirror no)
-			(drillshape 1)
+			(drillshape 0)
 			(scaleselection 1)
-			(outputdirectory "")
+			(outputdirectory "jlcpcb/")
 		)
 	)
@@
 			)
 		)
-		(property "Value" "DMN2991UFB4"
+		(property "Value" "DMN2300UFB4-7B"
 			(at 0 -1.6 0)
 			(layer "B.Fab")
