File: electronics/reward_port_2_sided/kicad/reward_port.kicad_pcb (KiCad board)
At the start: 4 copper layers, 30 x 21 mm, 59 parts, among them J1 SM04B-GHS-TB, J2 SM10B-GHS-TB, J3 SM10B-GHS-TB, J4 SM04B-GHS-TB, J5 Conn_SWD, J6 SM02B-GHS-TB, J7 SM02B-GHS-TB, Q1 2N7002PW, Q2 2N7002PW, Q3 2N7002PW, Q4 2N7002PW, U1 THVD1410DGKR, U2 THVD1410DGKR, U3 PAM8302AASCR, U4 STM32G071GBU6, U5 DRV8837

Commit message: reward port schematic update to support latching valve as an option
Parts:
- added R24: 10k, Resistor_SMD:R_0402_1005Metric, B.Cu at (79.1, 127.5)
- turned R23 to 0 degrees
Connections:
- R23 pad 1: /TIM1_CH1 -> GND
- R23 pad 2: GND -> /TIM1_CH1
- U4 pad 18: unconnected-(U4-PA11[PA9]-Pad18) -> /TIM1_CH2
- U5 pad 5: GND -> /TIM1_CH2
Routing:
- net /TIM1_CH2: track 0.00 -> 57.4 mm, vias 0 -> 4
- net /VLOAD: track 74.7 -> 78.5 mm
- net GND: track 88.3 -> 87.6 mm, vias 13 -> 14
