File: electronics/reward_port_2_sided/kicad/reward_port.kicad_sch (KiCad schematic)
At the start: 61 parts, among them J1 SM04B-GHS-TB, J2 SM10B-GHS-TB, J3 SM10B-GHS-TB, J4 SM04B-GHS-TB, J5 Conn_SWD, J6 SM02B-GHS-TB, J7 SM02B-GHS-TB, Q1 2N7002PW, Q2 2N7002PW, Q3 2N7002PW, Q4 2N7002PW, U1 THVD1410DGKR, U2 THVD1410DGKR, U3 PAM8302AASCR, U4 STM32G071GBU6, U5 DRV8837

Commit message: reward port schematic update to support latching valve as an option
Parts:
- added R24: 10k, Resistor_SMD:R_0402_1005Metric, symbol Device:R
Connections:
- net GND: now also R23.1, R24.1; no longer R23.2, U5.5 (IN2)
- net TIM1_CH1: now also R23.2; no longer R23.1
- net TIM1_CH2: now reaches U4.18 (PA11[PA9])
- net TIM1_CH2: now also U5.5 (IN2), R24.2
- no-connect marks 12 -> 11
Other:
- moved on the sheet: R23
